File: PCB_Roboshot/Roboshot/Roboshot.kicad_pcb (KiCad board)
At the start: 2 copper layers, 71.6 x 91.9 mm, 14 parts, among them J1 Conn_01x06, J10 Conn_01x04, J11 Conn_01x04, J2 Conn_01x02, J3 Conn_01x06, J4 Conn_01x04, J5 Conn_01x06, J6 Conn_01x06, J7 Conn_01x06, J8 Conn_01x02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

Commit message: Diseño terminado
Parts:
- removed J10: Conn_01x04, Connector_PinSocket_2.54mm:PinSocket_1x04_P2.54mm_Vertical_SMD_Pin1Right
- removed J11: Conn_01x04, Connector_PinSocket_2.54mm:PinSocket_1x04_P2.54mm_Vertical
- removed J4: Conn_01x04, Connector_PinHeader_2.54mm:PinHeader_1x04_P2.54mm_Vertical
- removed J6, J7: Conn_01x06, Connector_PinHeader_2.54mm:PinHeader_1x06_P2.54mm_Vertical
- removed J8: Conn_01x02, Connector_PinHeader_2.54mm:PinHeader_1x02_P2.54mm_Vertical
- added C1: C_Polarized, Capacitor_THT:CP_Radial_D8.0mm_P5.00mm, F.Cu at (245.5, 171.5)
- added HX711: DualChannel, DualChannel_HX711:Dual Channel, F.Cu at (298.0, 147.5)
- added J2: Conn_01x08, Connector_PinHeader_2.54mm:PinHeader_1x08_P2.54mm_Vertical, F.Cu at (227.3, 136.6)
- added LEDEXT.1: Conn_01x02, TerminalBlock:TerminalBlock_bornier-2_P5.08mm, F.Cu at (242.9, 194.3)
- added LEDSIGN1: Conn_01x03, Connector_JST:JST_EH_B3B-EH-A_1x03_P2.50mm_Vertical, F.Cu at (264.3, 196.0)
- added LIGHT1: Conn_01x02, TerminalBlock:TerminalBlock_bornier-2_P5.08mm, F.Cu at (229.7, 182.7)
- added LOGICLEVELSHIFTER1: 757, LogicLevel:MODULE_757, F.Cu at (289.8, 162.1)
- added OE1: Conn_01x02, Connector_PinHeader_2.54mm:PinHeader_1x02_P2.54mm_Vertical, F.Cu at (244.9, 124.8)
- added PCA9685: 815, PCA9685:PCA9685, F.Cu at (264.8, 165.4)
- added PUMP2: Conn_01x02, TerminalBlock:TerminalBlock_bornier-2_P5.08mm, F.Cu at (254.4, 113.1)
- added Q1_LIGHT1: BC546, Package_TO_SOT_THT:TO-92_Inline, F.Cu at (245.9, 156.4)
- added Q2_PUMP1: BC546, Package_TO_SOT_THT:TO-92_Inline, F.Cu at (249.8, 131.6)
- added R2: R, Resistor_SMD:R_0805_2012Metric, F.Cu at (242.4, 137.4)
- added R3: R, Resistor_SMD:R_0805_2012Metric, F.Cu at (243.8, 150.5)
- added R4: R, Resistor_SMD:R_0805_2012Metric, F.Cu at (251.1, 140.3)
- added R5: R, Resistor_SMD:R_0805_2012Metric, F.Cu at (243.4, 147.0)
- ExternalSource1: renamed from J9; footprint Connector_BarrelJack:BarrelJack_GCT_DCJ200-10-A_Horizontal -> Connector_BarrelJack:BarrelJack_Horizontal
- J1, J5: value Conn_01x06 -> Conn_01x01; footprint Connector_PinHeader_2.54mm:PinHeader_1x06_P2.54mm_Vertical -> Connector_PinHeader_2.54mm:PinHeader_1x01_P2.54mm_Vertical
- J3: value Conn_01x06 -> Conn_01x04; footprint Connector_PinHeader_2.54mm:PinHeader_1x06_P2.54mm_Vertical -> Connector_PinHeader_2.54mm:PinHeader_1x04_P2.54mm_Vertical
- U1: footprint Rubilon:3M_7840-0000PR -> Connector_IDC:IDC-Header_2x20_P2.54mm_Vertical
- moved G1 53.2 mm to (293.5, 194.3)
- moved J5 39.4 mm to (256.8, 156.9), turned to 0 degrees
- moved R1 36.7 mm to (269.7, 188.6), turned to 180 degrees
- moved J3 29.0 mm to (283.1, 112.2)
- moved J1 19.1 mm to (256.8, 153.6), turned to 0 degrees
- moved U1 9.02 mm to (233.9, 123.8), turned to 0 degrees
- moved ExternalSource1 6.19 mm to (287.5, 182.2), turned to 180 degrees
- moved PUMP1 5.58 mm to (271.4, 113.4), turned to 180 degrees
- renumbered J2 to PUMP1
Connections:
- J5 pad 1: unconnected-(J5-Pad1) -> +5VA
- PUMP1 pad 1: /GPIO24(GEN5) -> /HV1
Routing:
- net /GPIO19(SPI1_MISO): track 0.00 -> 137.9 mm, vias 0 -> 3
- net +5VA: track 101.1 -> 206.6 mm
- net /GPIO24(GEN5): track 43.7 -> 148.5 mm, vias 0 -> 1
- net /HV1: track 0.00 -> 82.8 mm
- net /HV2: track 115.0 -> 40.4 mm
- net GND: track 224.5 -> 290.7 mm
- net /HV3: track 0.00 -> 60.2 mm
- net Net-(PCA9685-PadV+_1): track 0.00 -> 58.2 mm
- net Net-(PCA9685-PadOE_1): track 0.00 -> 58.2 mm
- net /LIGHT: track 0.00 -> 52.8 mm
- net /GPIO2(SDA1): track 60.6 -> 112.7 mm
- net /GPIO3(SCL1): track 70.9 -> 112.9 mm
- net +3V3: track 120.6 -> 162.3 mm
- net /A+: track 11.8 -> 49.0 mm
- net +5V: track 103.0 -> 68.4 mm, vias 0 -> 1
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Other:
- board size 71.6 x 91.9 mm -> 78.3 x 91.9 mm
- board text added: "A+"
- board text added: "A-"
- board text added: "E+"
- board text added: "E-"

Commit message: Placa finalizada
Parts:
- moved PUMP1 1.39 mm to (270.0, 113.6)
- moved G1 0.71 mm to (294.2, 194.3)
Connections:
- LOGICLEVELSHIFTER1 pad GND: (no net) -> GND
Routing:
- net GND: track 290.7 -> 287.6 mm
- net /HV1: track 82.8 -> 84.1 mm
- added copper zone on B.Cu, net GND
- added copper zone on F.Cu, net GND

Commit message: Placa_roboshot
Parts:
- removed ExternalSource1: Conn_01x02, Connector_BarrelJack:BarrelJack_Horizontal
- removed LOGICLEVELSHIFTER1: 757, LogicLevel:MODULE_757
- removed PUMP1, PUMP2: Conn_01x02, TerminalBlock:TerminalBlock_bornier-2_P5.08mm
- removed Q2_PUMP1: BC546, Package_TO_SOT_THT:TO-92_Inline
- added C2: C_Polarized, Capacitor_THT:CP_Radial_D8.0mm_P5.00mm, F.Cu at (256.1, 171.1)
- added E.lSource1: Conn_01x02, Connector_BarrelJack:BarrelJack_Horizontal, F.Cu at (291.7, 185.2)
- added LEDEXT.2: Conn_01x02, TerminalBlock:TerminalBlock_bornier-2_P5.08mm, F.Cu at (297.7, 125.7)
- added LEDSIGN2: Conn_01x03, Connector_JST:JST_EH_B3B-EH-A_1x03_P2.50mm_Vertical, F.Cu at (286.0, 126.0)
- added LOGIC_LEVEL_SHIFTER1: Logic_Level_Shifter, Elevador:Elevador_voltaje, F.Cu at (280.2, 136.0)
- added PUMP_AC1: Conn_01x02, TerminalBlock:TerminalBlock_bornier-2_P5.08mm, F.Cu at (297.8, 157.6)
- added PUMP_DC1: Conn_01x02, TerminalBlock:TerminalBlock_bornier-2_P5.08mm, F.Cu at (297.7, 171.0)
- added Q2_PUMP_DC1: BC546, Package_TO_SOT_THT:TO-92_Inline, F.Cu at (286.3, 174.2)
- added R6: R, Resistor_SMD:R_0805_2012Metric, F.Cu at (280.0, 130.1)
- moved J3 94.2 mm to (240.7, 196.2)
- moved LEDEXT.1 75.8 mm to (297.8, 142.0), turned to -90 degrees
- moved HX711 66.4 mm to (255.0, 198.0), turned to 0 degrees
- moved G1 61.8 mm to (232.4, 191.7)
- moved LIGHT1 58.8 mm to (284.9, 162.4), turned to 90 degrees
- moved LEDSIGN1 58.3 mm to (286.8, 142.2), turned to -90 degrees
- moved R1 45.6 mm to (280.6, 144.3), turned to 0 degrees
- moved PCA9685 34.9 mm to (237.0, 144.2), turned to -90 degrees
- moved R5 34.5 mm to (268.1, 171.0)
- moved J2 32.0 mm to (256.6, 123.6), turned to 90 degrees
- moved R3 31.4 mm to (273.0, 161.9)
- moved Q1_LIGHT1 27.5 mm to (273.4, 156.2), turned to 90 degrees
- moved C1 19.3 mm to (256.9, 156.0)
- moved OE1 18.1 mm to (230.0, 114.5), turned to 0 degrees
- moved R4 14.7 mm to (263.9, 147.5), turned to 0 degrees
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Connections:
- R2 pad 1: /GPIO23(GEN4) -> /GPIO25(GEN6)
Routing:
- net /GPIO19(SPI1_MISO): track 137.9 -> 38.4 mm, vias 3 -> 0
- net +5V: track 68.4 -> 159.8 mm, vias 1 -> 0
- net /GPIO25(GEN6): track 0.00 -> 89.0 mm, vias 0 -> 1
- net /GPIO24(GEN5): track 148.5 -> 75.4 mm, vias 1 -> 0
- net /GPIO12(PWM0): track 0.00 -> 63.7 mm
- net +3V3: track 162.3 -> 107.3 mm
- net /HV3: track 60.2 -> 6.26 mm
- net /HV1: track 84.1 -> 38.4 mm, vias 0 -> 1
- net /LIGHT: track 52.8 -> 12.1 mm
- net /A+: track 49.0 -> 8.93 mm
- net /GPIO3(SCL1): track 112.9 -> 73.0 mm
- net /A-: track 52.9 -> 13.2 mm
- net /E-: track 56.4 -> 17.1 mm
- net /GPIO2(SDA1): track 112.7 -> 73.6 mm
- net /E+: track 58.4 -> 21.4 mm
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