File: PCB_Roboshot/Roboshot/Roboshot.kicad_sch (KiCad schematic)
At the start: 14 parts, among them J1 Conn_01x06, J10 Conn_01x04, J2 Conn_01x02, J3 Conn_01x06, J4 Conn_01x04, J5 Conn_01x06, J6 Conn_01x06, J7 Conn_01x06, J8 Conn_01x02, J9 Conn_01x02, U1 7840-0000PR

Commit message: Diseño terminado
Parts:
- removed J1, J3, J5, J6, J7: Conn_01x06, Connector_PinHeader_2.54mm:PinHeader_1x06_P2.54mm_Vertical, symbol Connector_Generic:Conn_01x06
- removed J10: Conn_01x04, Connector_PinSocket_2.54mm:PinSocket_1x04_P2.54mm_Vertical_SMD_Pin1Right, symbol Connector_Generic:Conn_01x04
- removed J4: Conn_01x04, Connector_PinHeader_2.54mm:PinHeader_1x04_P2.54mm_Vertical, symbol Connector_Generic:Conn_01x04
- removed J8: Conn_01x02, Connector_PinHeader_2.54mm:PinHeader_1x02_P2.54mm_Vertical, symbol Connector_Generic:Conn_01x02
- added C1: C_Polarized, Capacitor_THT:CP_Radial_D8.0mm_P5.00mm, symbol Device:C_Polarized
- added HX711: DualChannel, DualChannel_HX711:Dual Channel, symbol DualChannel_HX711:DualChannel
- added J1, J5: Conn_01x01, Connector_PinHeader_2.54mm:PinHeader_1x01_P2.54mm_Vertical, symbol Connector_Generic:Conn_01x01
- added J2: Conn_01x08, Connector_PinHeader_2.54mm:PinHeader_1x08_P2.54mm_Vertical, symbol Connector_Generic:Conn_01x08
- added J3: Conn_01x04, Connector_PinHeader_2.54mm:PinHeader_1x04_P2.54mm_Vertical, symbol Connector_Generic:Conn_01x04
- added LIGHT1, PUMP2: Conn_01x02, TerminalBlock:TerminalBlock_bornier-2_P5.08mm, symbol Connector_Generic:Conn_01x02
- added LOGIC_LEVEL_SHIFTER1: Logic_Level_Shifter, LogicLevel:MODULE_757, symbol Logic_level:Logic_Level_Shifter
- added OE1: Conn_01x02, Connector_PinHeader_2.54mm:PinHeader_1x02_P2.54mm_Vertical, symbol Connector_Generic:Conn_01x02
- added PCA9685: 815, PCA9685:PCA9685, symbol PCA9685:815
- added Q1_LIGHT1, Q2_PUMP1: BC546, Package_TO_SOT_THT:TO-92_Inline, symbol Transistor_BJT:BC546
- added R2, R3, R4, R5: R, Resistor_SMD:R_0805_2012Metric, symbol Device:R
- ExternalSource1: renamed from J9; footprint Connector_BarrelJack:BarrelJack_GCT_DCJ200-10-A_Horizontal -> Connector_BarrelJack:BarrelJack_Horizontal
- LEDEXT.1: renamed from J?; footprint (none) -> TerminalBlock:TerminalBlock_bornier-2_P5.08mm
- LEDSIGN1: renamed from J?; footprint (none) -> Connector_JST:JST_EH_B3B-EH-A_1x03_P2.50mm_Vertical
- U1: footprint Rubilon:3M_7840-0000PR -> Connector_IDC:IDC-Header_2x20_P2.54mm_Vertical
- renumbered J2 to PUMP1
Connections:
- net +3V3: now also LOGIC_LEVEL_SHIFTER1.LV, PCA9685.VCC_1 (VCC), PCA9685.VCC_2 (VCC)
- net +5V: now also HX711.VCC
- net +5VA: now also C1.1, J5.1 (Pin_1), LIGHT1.1 (Pin_1), LOGIC_LEVEL_SHIFTER1.HV, PUMP2.1 (Pin_1)
- net A+: now also HX711.A+, J3.4 (Pin_4)
- net A-: now also HX711.A-, J3.3 (Pin_3)
- net E+: now also HX711.E+, J3.1 (Pin_1)
- net E-: now also HX711.E-, J3.2 (Pin_2)
- net GND: now also C1.2, HX711.GND, J1.1 (Pin_1), LOGIC_LEVEL_SHIFTER1.GND, OE1.2 (Pin_2), PCA9685.GND_1 (GND), PCA9685.GND_10 (GND), PCA9685.GND_11 (GND), PCA9685.GND_12 (GND), PCA9685.GND_13 (GND), PCA9685.GND_14 (GND), PCA9685.GND_15 (GND), PCA9685.GND_16 (GND), PCA9685.GND_17 (GND), PCA9685.GND_18 (GND), PCA9685.GND_2 (GND), PCA9685.GND_3 (GND), PCA9685.GND_4 (GND), PCA9685.GND_5 (GND), PCA9685.GND_6 (GND), PCA9685.GND_7 (GND), PCA9685.GND_8 (GND), PCA9685.GND_9 (GND), R3.1, R5.1
- net GPIO10(SPI0_MOSI): now also J2.4 (Pin_4)
- net GPIO11(SPI0_SCK): now also J2.6 (Pin_6)
- net GPIO13(PWM1): now also J2.8 (Pin_8)
- net GPIO17(GEN0): now also J2.1 (Pin_1)
- net GPIO18(GEN1)(PWM0): now also LOGIC_LEVEL_SHIFTER1.LV2
- net GPIO19(SPI1_MISO): now also LOGIC_LEVEL_SHIFTER1.LV3
- net GPIO2(SDA1): now also PCA9685.SDA_1 (SDA), PCA9685.SDA_2 (SDA)
- net GPIO20(SPI1_MOSI): now also HX711.SCK
- net GPIO21(SPI1_SCK): now also HX711.DT
- net GPIO22(GEN3): now also J2.3 (Pin_3)
- net GPIO23(GEN4): now also OE1.1 (Pin_1), R2.1
- net GPIO24(GEN5): now also LOGIC_LEVEL_SHIFTER1.LV1; no longer PUMP1.1 (Pin_1)
- net GPIO27(GEN2): now also J2.2 (Pin_2)
- net GPIO3(SCL1): now also PCA9685.SCL_1 (SCL), PCA9685.SCL_2 (SCL)
- net GPIO9(SPI0_MISO): now also J2.5 (Pin_5)
- net HV1: now also PUMP1.1 (Pin_1), LOGIC_LEVEL_SHIFTER1.HV1
- net HV2: now also LOGIC_LEVEL_SHIFTER1.HV2
- net HV3: now also LOGIC_LEVEL_SHIFTER1.HV3, R4.1
- net HV4: now also LOGIC_LEVEL_SHIFTER1.HV4
- net ID_SD: now also J2.7 (Pin_7)
- net LV4: now also LOGIC_LEVEL_SHIFTER1.LV4
- new net: Q1_LIGHT1.2 (B), R2.2
- new net: Q2_PUMP1.3 (E), R5.2
- new net: Q1_LIGHT1.3 (E), R3.2
- new net: PCA9685.OE_1 (~{OE}), PCA9685.OE_2 (~{OE})
- new net: PCA9685.V+_1 (V+), PCA9685.V+_10 (V+), PCA9685.V+_11 (V+), PCA9685.V+_12 (V+), PCA9685.V+_13 (V+), PCA9685.V+_14 (V+), PCA9685.V+_15 (V+), PCA9685.V+_16 (V+), PCA9685.V+_17 (V+), PCA9685.V+_18 (V+), PCA9685.V+_2 (V+), PCA9685.V+_3 (V+), PCA9685.V+_4 (V+), PCA9685.V+_5 (V+), PCA9685.V+_6 (V+), PCA9685.V+_7 (V+), PCA9685.V+_8 (V+), PCA9685.V+_9 (V+)
- new net: Q2_PUMP1.2 (B), R4.2
- new net LIGHT: LIGHT1.2 (Pin_2), Q1_LIGHT1.1 (C)
- new net PUMP: PUMP2.2 (Pin_2), Q2_PUMP1.1 (C)
Other:
- note added: "ADICIONALES"
- note added: "BOMBA DE SUCCIÓN"
- note added: "LUZ DE ALARMA"
- note added: "POLOLU A4988"
- note removed: "BORNERA"
- moved on the sheet: ExternalSource1, LEDEXT.1, LEDSIGN1, PUMP1, R1, U1

Commit message: Placa_roboshot
Parts:
- added C2: C_Polarized, Capacitor_THT:CP_Radial_D8.0mm_P5.00mm, symbol Device:C_Polarized
- added LEDEXT.2: Conn_01x02, TerminalBlock:TerminalBlock_bornier-2_P5.08mm, symbol Connector_Generic:Conn_01x02
- added LEDSIGN2: Conn_01x03, Connector_JST:JST_EH_B3B-EH-A_1x03_P2.50mm_Vertical, symbol Connector_Generic:Conn_01x03
- added R6: R, Resistor_SMD:R_0805_2012Metric, symbol Device:R
- LOGIC_LEVEL_SHIFTER1: footprint LogicLevel:MODULE_757 -> Elevador:Elevador_voltaje
- renumbered PUMP1 to PUMP_AC1, PUMP2 to PUMP_DC1, Q2_PUMP1 to Q2_PUMP_DC1
Connections:
- net LV4 is gone; now on net GPIO12(PWM0): LOGIC_LEVEL_SHIFTER1.LV4
- net +5VA: now also C2.1, LEDEXT.2.2 (Pin_2), LEDSIGN2.3 (Pin_3)
- net GND: now also C2.2, LEDEXT.2.1 (Pin_1), LEDSIGN2.1 (Pin_1)
- net GPIO23(GEN4): no longer R2.1
- net GPIO25(GEN6): now also R2.1
- net HV4: now also R6.1
- new net: LEDSIGN2.2 (Pin_2), R6.2
Other:
- moved on the sheet: OE1
