File: PCB_Roboshot/Roboshot/Roboshot.kicad_sch (KiCad schematic)
At the start: 29 parts, among them J2 Conn_01x08, J4 Conn_01x03, J6 Conn_01x04, Q1_LIGHT1 BC546, Q1_PCA1 BC546, Q2_PUMP_DC1 BC546, U1 7840-0000PR, U2 H

Commit message: Placa final_Roboshot
Parts:
- removed P.Button1: Conn_01x02, Connector_PinHeader_2.54mm:PinHeader_1x02_P2.54mm_Vertical, symbol Connector_Generic:Conn_01x02
- removed Q1_PCA1, Q2_PUMP_DC1: BC546, Package_TO_SOT_THT:TO-92_Inline, symbol Transistor_BJT:BC546
- removed R3: R, Resistor_SMD:R_0805_2012Metric, symbol Device:R
- added B.OUTPUT1, BUTTON1, Q_PCA9685: BC546, Package_TO_SOT_THT:TO-92_Inline, symbol Transistor_BJT:BC546
- added D1: LED, LED_THT:LED_D3.0mm, symbol Device:LED
- added IRFZ44N1: BSP89, Package_TO_SOT_THT:SIPAK_Vertical, symbol Transistor_FET:BSP89
- added R10, R9: R, Resistor_SMD:R_0805_2012Metric, symbol Device:R
- added SW1: SW_Push_Dual_x2, Connector_PinHeader_2.54mm:PinHeader_1x02_P2.54mm_Vertical, symbol Switch:SW_Push_Dual_x2
Connections:
- net GND_PCA9685 is gone; now on net GND: PCA9685.GND_1 (GND), PCA9685.GND_10 (GND), PCA9685.GND_11 (GND), PCA9685.GND_12 (GND), PCA9685.GND_13 (GND), PCA9685.GND_14 (GND), PCA9685.GND_15 (GND), PCA9685.GND_16 (GND), PCA9685.GND_17 (GND), PCA9685.GND_18 (GND), PCA9685.GND_2 (GND), PCA9685.GND_3 (GND), PCA9685.GND_4 (GND), PCA9685.GND_5 (GND), PCA9685.GND_6 (GND), PCA9685.GND_7 (GND), PCA9685.GND_8 (GND), PCA9685.GND_9 (GND)
- net +3V3: no longer PCA9685.VCC_1 (VCC), PCA9685.VCC_2 (VCC)
- net +5V: now also PCA9685.VCC_1 (VCC), PCA9685.VCC_2 (VCC), Q1_LIGHT1.1 (C), R5.1, Q_PCA9685.1 (C), R10.2; no longer LIGHT1.1 (Pin_1), PCA9685.V+_1 (V+), PCA9685.V+_10 (V+), PCA9685.V+_11 (V+), PCA9685.V+_12 (V+), PCA9685.V+_13 (V+), PCA9685.V+_14 (V+), PCA9685.V+_15 (V+), PCA9685.V+_16 (V+), PCA9685.V+_17 (V+), PCA9685.V+_18 (V+), PCA9685.V+_2 (V+), PCA9685.V+_3 (V+), PCA9685.V+_4 (V+), PCA9685.V+_5 (V+), PCA9685.V+_6 (V+), PCA9685.V+_7 (V+), PCA9685.V+_8 (V+), PCA9685.V+_9 (V+)
- net GND: now also LIGHT1.2 (Pin_2), R4.2, B.OUTPUT1.3 (E), BUTTON1.3 (E), D1.1 (K), IRFZ44N1.3 (S); no longer R5.1, R8.1
- net GPIO12(PWM0): now also LOGIC_LEVEL_SHIFTER1.LV1; no longer LOGIC_LEVEL_SHIFTER1.LV4
- net GPIO14(TXD0): now also R8.1, R9.1
- net GPIO18(GEN1)(PWM0): now also LOGIC_LEVEL_SHIFTER1.LV3; no longer LOGIC_LEVEL_SHIFTER1.LV2
- net GPIO19(SPI1_MISO): now also LOGIC_LEVEL_SHIFTER1.LV2; no longer LOGIC_LEVEL_SHIFTER1.LV3
- net GPIO22(GEN3): no longer R7.1
- net GPIO24(GEN5): now also LOGIC_LEVEL_SHIFTER1.LV4; no longer LOGIC_LEVEL_SHIFTER1.LV1
- net GPIO26: now also R7.1
- net GPIO3(SCL1): now also SW1.1 (C)
- net HV1: now also R1.1; no longer J4.1 (Pin_1)
- net HV2: now also R4.1, IRFZ44N1.1 (G); no longer R1.1
- net HV3: now also R6.1; no longer R4.1
- net HV4: now also J4.1 (Pin_1); no longer R6.1
- net LIGHT: now also LIGHT1.1 (Pin_1), Q1_LIGHT1.3 (E); no longer LIGHT1.2 (Pin_2), Q1_LIGHT1.1 (C)
- net PUMP: now also IRFZ44N1.2 (D)
- net at R5.2: now also B.OUTPUT1.2 (B)
- net at R7.2: now also Q_PCA9685.2 (B)
- net at R8.2: now also BUTTON1.2 (B)
- new net: BUTTON1.1 (C), R10.1
- new net: D1.2 (A), R9.2
- new net 2N_PCA9685: PCA9685.V+_1 (V+), PCA9685.V+_10 (V+), PCA9685.V+_11 (V+), PCA9685.V+_12 (V+), PCA9685.V+_13 (V+), PCA9685.V+_14 (V+), PCA9685.V+_15 (V+), PCA9685.V+_16 (V+), PCA9685.V+_17 (V+), PCA9685.V+_18 (V+), PCA9685.V+_2 (V+), PCA9685.V+_3 (V+), PCA9685.V+_4 (V+), PCA9685.V+_5 (V+), PCA9685.V+_6 (V+), PCA9685.V+_7 (V+), PCA9685.V+_8 (V+), PCA9685.V+_9 (V+), Q_PCA9685.3 (E)
- new net Button_OUTPUT: B.OUTPUT1.1 (C), SW1.2 (D)
Other:
- note added: "LED INDICADOR"
- moved on the sheet: Ext.Source1, J2, J4, J6, LIGHT1, OE1, PCA9685, PUMP_DC1, Q1_LIGHT1, R2, R4, R7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

Commit message: revision de PCB
Parts:
- IRFZ44N1: footprint Package_TO_SOT_THT:SIPAK_Vertical -> Package_TO_SOT_THT:TO-220F-3_Horizontal_TabDown
- renumbered J2 to J1, J6 to LoadCell1, PCA9685 to PCA1, Q_PCA9685 to Q_PCA1, R2 to R1, R4 to R2, R7 to R3, R1 to R4, R6 to R5, R5 to R6, R8 to R7, R9 to R8, R10 to R9, J4 to SCR1
Connections:
- net +3V3: now also U1.1
- net +5V: now also PUMP_DC1.2 (Pin_2); no longer PUMP_DC1.1 (Pin_1)
- net GND: now also LIGHT1.1 (Pin_1), U1.14, U1.20, U1.25, U1.30, U1.34, U1.6, U1.9; no longer LIGHT1.2 (Pin_2)
- net HV1: now also LOGIC_LEVEL_SHIFTER1.HV3; no longer LOGIC_LEVEL_SHIFTER1.HV1
- net HV3: now also LOGIC_LEVEL_SHIFTER1.HV4; no longer LOGIC_LEVEL_SHIFTER1.HV3
- net HV4: now also LOGIC_LEVEL_SHIFTER1.HV1; no longer LOGIC_LEVEL_SHIFTER1.HV4
- net LIGHT: now also LIGHT1.2 (Pin_2); no longer LIGHT1.1 (Pin_1)
- net PUMP: now also PUMP_DC1.1 (Pin_1); no longer PUMP_DC1.2 (Pin_2)
Other:
- moved on the sheet: B.OUTPUT1, BUTTON1, C1, C2, Ext.Source1, IRFZ44N1, J1, LEDEXT.1, LEDEXT.2, LEDSIGN1, LEDSIGN2, LIGHT1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
