File: PCB_Roboshot/Roboshot/Roboshot.kicad_sch (KiCad schematic)
At the start: 33 parts, among them J1 Conn_01x08, Q1_LIGHT1 BC546, SW1 SW_Push_Dual_x2, U1 7840-0000PR, U2 H

Commit message: Defini Valores en resistencia y arregle el problema el InvPin en el boton de Power
Parts:
- R1: value R -> 4,7K
- R2: value R -> 10K
- R3, R6, R7: value R -> 4K7
- R4, R5, R8: value R -> 330
Connections:
- net +5V: no longer R6.1
- net Inv.OUPUT: now reaches BUTTON1.1 (C), R9.1
- net Inv.OUPUT: now also R6.1
Changed lines of the file:
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@@
   (junction (at 47.752 65.532) (diameter 0) (color 0 0 0 0)
   )
+  (junction (at 262.128 48.26) (diameter 0) (color 0 0 0 0)
+  )
   (junction (at 47.752 52.832) (diameter 0) (color 0 0 0 0)
   )
@@
   (junction (at 90.17 70.612) (diameter 0) (color 0 0 0 0)
   )
-  (junction (at 272.542 48.26) (diameter 0) (color 0 0 0 0)
-  )
   (junction (at 38.1 35.052) (diameter 0) (color 0 0 0 0)
   )
@@
     (stroke (width 0) (type default) (color 0 0 0 0))
   )
-  (wire (pts (xy 263.144 48.26) (xy 257.81 48.26))
+  (wire (pts (xy 263.144 48.26) (xy 262.128 48.26))
     (stroke (width 0) (type default) (color 0 0 0 0))
   )
@@
     (stroke (width 0) (type default) (color 0 0 0 0))
   )
-  (wire (pts (xy 272.542 48.26) (xy 274.066 48.26))
-    (stroke (width 0) (type default) (color 0 0 0 0))
-  )
   (wire (pts (xy 36.83 37.592) (xy 50.8 37.592))
     (stroke (width 0) (type default) (color 0 0 0 0))
@@
     (stroke (width 0) (type default) (color 0 0 0 0))
   )
+  (wire (pts (xy 262.128 48.26) (xy 257.81 48.26))
+    (stroke (width 0) (type default) (color 0 0 0 0))
+  )
   (wire (pts (xy 229.87 118.364) (xy 236.22 118.364))
     (stroke (width 0) (type default) (color 0 0 0 0))
@@
     (stroke (width 0) (type default) (color 0 0 0 0))
   )
+  (wire (pts (xy 262.128 48.26) (xy 262.128 50.8))
+    (stroke (width 0) (type default) (color 0 0 0 0))
+  )
   (wire (pts (xy 237.236 158.75) (xy 234.696 158.75))
     (stroke (width 0) (type default) (color 0 0 0 0))
@@
     (stroke (width 0) (type default) (color 0 0 0 0))
   )
-  (wire (pts (xy 272.542 48.26) (xy 272.542 52.07))
-    (stroke (width 0) (type default) (color 0 0 0 0))
-  )
   (wire (pts (xy 36.83 57.912) (xy 50.8 57.912))
     (stroke (width 0) (type default) (color 0 0 0 0))
@@
     (stroke (width 0) (type default) (color 0 0 0 0))
   )
-  (wire (pts (xy 270.764 48.26) (xy 272.542 48.26))
+  (wire (pts (xy 270.764 48.26) (xy 274.066 48.26))
     (stroke (width 0) (type default) (color 0 0 0 0))
   )
@@
     (effects (font (size 1.27 1.27)) (justify left bottom))
   )
-  (label "Inv.OUPUT" (at 272.542 52.07 270)
+  (label "Inv.OUPUT" (at 262.128 50.8 270)
     (effects (font (size 1.27 1.27)) (justify right bottom))
   )
@@
   (symbol (lib_id "Transistor_FET:BSP89") (at 173.99 122.428 0) (unit 1)
     (in_bom yes) (on_board yes) (fields_autoplaced)
-    (property "Reference" "IRFZ44N1" (id 0) (at 179.832 121.1579 0)
-      (effects (font (size 1.27 1.27)) (justify left))
-    )
-    (property "Value" "BSP89" (id 1) (at 179.832 123.6979 0)
+    (property "Reference" "IRFZ44N1" (id 0) (at 180.34 121.1579 0)
+      (effects (font (size 1.27 1.27)) (justify left))
+    )
+    (property "Value" "BSP89" (id 1) (at 180.34 123.6979 0)
       (effects (font (size 1.27 1.27)) (justify left))
     )
@@
     (in_bom yes) (on_board yes) (fields_autoplaced)
     (property "Reference" "R1" (id 0) (at 111.379 113.792 90))
-    (property "Value" "R" (id 1) (at 111.379 116.332 90))
+    (property "Value" "4,7K" (id 1) (at 111.379 116.332 90))
     (property "Footprint" "Resistor_SMD:R_0805_2012Metric" (id 2) (at 111.379 121.92 90)
       (effects (font (size 1.27 1.27)) hide)
@@
     (in_bom yes) (on_board yes)
     (property "Reference" "R7" (id 0) (at 243.586 51.054 90))
-    (property "Value" "R" (id 1) (at 243.586 53.086 90))
+    (property "Value" "4K7" (id 1) (at 243.586 53.086 90))
     (property "Footprint" "Resistor_SMD:R_0805_2012Metric" (id 2) (at 243.586 57.15 90)
       (effects (font (size 1.27 1.27)) hide)
@@
   (symbol (lib_id "Device:R") (at 226.06 118.364 90) (unit 1)
     (in_bom yes) (on_board yes) (fields_autoplaced)
-    (property "Reference" "R4" (id 0) (at 226.06 112.014 90))
-    (property "Value" "R" (id 1) (at 226.06 114.554 90))
+    (property "Reference" "R4" (id 0) (at 226.06 111.76 90))
+    (property "Value" "330" (id 1) (at 226.06 114.3 90))
     (property "Footprint" "Resistor_SMD:R_0805_2012Metric" (id 2) (at 226.06 120.142 90)
       (effects (font (size 1.27 1.27)) hide)
@@
     (in_bom yes) (on_board yes)
     (property "Reference" "R6" (id 0) (at 243.078 71.628 90))
-    (property "Value" "R" (id 1) (at 243.078 73.66 90))
+    (property "Value" "4K7" (id 1) (at 243.078 73.66 90))
     (property "Footprint" "Resistor_SMD:R_0805_2012Metric" (id 2) (at 243.078 77.724 90)
       (effects (font (size 1.27 1.27)) hide)
@@
   (symbol (lib_id "Device:R") (at 249.428 29.972 90) (unit 1)
     (in_bom yes) (on_board yes) (fields_autoplaced)
-    (property "Reference" "R8" (id 0) (at 249.428 23.876 90))
-    (property "Value" "R" (id 1) (at 249.428 26.416 90))
+    (property "Reference" "R8" (id 0) (at 249.428 24.13 90))
+    (property "Value" "330" (id 1) (at 249.428 26.67 90))
     (property "Footprint" "Resistor_SMD:R_0805_2012Metric" (id 2) (at 249.428 31.75 90)
       (effects (font (size 1.27 1.27)) hide)
@@
     (in_bom yes) (on_board yes) (fields_autoplaced)
     (property "Reference" "R5" (id 0) (at 227.076 139.7 90))
-    (property "Value" "R" (id 1) (at 227.076 142.24 90))
+    (property "Value" "330" (id 1) (at 227.076 142.24 90))
     (property "Footprint" "Resistor_SMD:R_0805_2012Metric" (id 2) (at 227.076 147.828 90)
       (effects (font (size 1.27 1.27)) hide)
@@
   )
   (symbol (lib_id "Transistor_BJT:BC546") (at 255.27 55.372 0) (unit 1)
-    (in_bom yes) (on_board yes) (fields_autoplaced)
-    (property "Reference" "BUTTON1" (id 0) (at 260.858 54.1019 0)
-      (effects (font (size 1.27 1.27)) (justify left))
-    )
-    (property "Value" "BC546" (id 1) (at 260.858 56.6419 0)
+    (in_bom yes) (on_board yes)
+    (property "Reference" "BUTTON1" (id 0) (at 244.602 58.166 0)
+      (effects (font (size 1.27 1.27)) (justify left))
+    )
+    (property "Value" "BC546" (id 1) (at 244.856 60.198 0)
       (effects (font (size 1.27 1.27)) (justify left))
     )
@@
     (in_bom yes) (on_board yes)
     (property "Reference" "R2" (id 0) (at 170.18 125.984 90))
-    (property "Value" "R" (id 1) (at 170.18 127.762 90))
+    (property "Value" "10K" (id 1) (at 170.18 127.762 90))
     (property "Footprint" "Resistor_SMD:R_0805_2012Metric" (id 2) (at 170.18 131.826 90)
       (effects (font (size 1.27 1.27)) hide)
@@
     (in_bom yes) (on_board yes) (fields_autoplaced)
     (property "Reference" "R3" (id 0) (at 187.452 48.768 90))
-    (property "Value" "R" (id 1) (at 187.452 51.308 90))
+    (property "Value" "4K7" (id 1) (at 187.452 51.308 90))
     (property "Footprint" "Resistor_SMD:R_0805_2012Metric" (id 2) (at 187.452 56.896 90)
       (effects (font (size 1.27 1.27)) hide)
@@
     )
     (path "/13bd04c7-596a-4201-b8df-dda405053e99"
-      (reference "R1") (unit 1) (value "R") (footprint "Resistor_SMD:R_0805_2012Metric")
+      (reference "R1") (unit 1) (value "4,7K") (footprint "Resistor_SMD:R_0805_2012Metric")
     )
     (path "/ece0afd5-7ecc-42fb-bb24-ee8d2e3730ff"
-      (reference "R2") (unit 1) (value "R") (footprint "Resistor_SMD:R_0805_2012Metric")
+      (reference "R2") (unit 1) (value "10K") (footprint "Resistor_SMD:R_0805_2012Metric")
     )
     (path "/ede0e183-80f6-494e-80cd-ed2cf77df68f"
-      (reference "R3") (unit 1) (value "R") (footprint "Resistor_SMD:R_0805_2012Metric")
+      (reference "R3") (unit 1) (value "4K7") (footprint "Resistor_SMD:R_0805_2012Metric")
     )
     (path "/3d0ffb99-3fe7-4b74-a599-53e7042a1c2e"
-      (reference "R4") (unit 1) (value "R") (footprint "Resistor_SMD:R_0805_2012Metric")
+      (reference "R4") (unit 1) (value "330") (footprint "Resistor_SMD:R_0805_2012Metric")
     )
     (path "/d08f9431-ef8a-42b7-a850-bcd8bb770f1b"
-      (reference "R5") (unit 1) (value "R") (footprint "Resistor_SMD:R_0805_2012Metric")
+      (reference "R5") (unit 1) (value "330") (footprint "Resistor_SMD:R_0805_2012Metric")
     )
     (path "/96c82320-024c-4ec3-a289-4346220e87f4"
-      (reference "R6") (unit 1) (value "R") (footprint "Resistor_SMD:R_0805_2012Metric")
+      (reference "R6") (unit 1) (value "4K7") (footprint "Resistor_SMD:R_0805_2012Metric")
     )
     (path "/345faa35-0c58-48d0-881b-ff3f1f050272"
-      (reference "R7") (unit 1) (value "R") (footprint "Resistor_SMD:R_0805_2012Metric")
+      (reference "R7") (unit 1) (value "4K7") (footprint "Resistor_SMD:R_0805_2012Metric")
     )
     (path "/cb9bb4c3-e2ef-4e82-8f8a-7c071851b70a"
-      (reference "R8") (unit 1) (value "R") (footprint "Resistor_SMD:R_0805_2012Metric")
+      (reference "R8") (unit 1) (value "330") (footprint "Resistor_SMD:R_0805_2012Metric")
     )
     (path "/948f2358-7454-481e-ad10-08a75434d4bb"
